File: boards/H-Bridge/brushed_v2.kicad_sch (KiCad schematic)
At the start: 14 parts, among them IC1 TC1108-3.3VDBTR, J1 Prog_Header, J2 CANBus, J3 UART, J4 Encoder, U1 STM32F103C8Tx

Commit message: Moved components to EVC lib
Parts:
- removed IC1: TC1108-3.3VDBTR, SOT230P700X180-4N, symbol SamacSys_Parts:TC1108-3.3VDBTR
- removed VR1: Throttle Potentiometer, P120PKY25BR10K, symbol Kicad_sym:P120PK-Y25BR10K
- added IC1: TC1108-3.3VDBTR, SOT230P700X180-4N, symbol Regulators:TC1108-3.3VDBTR
- added RV1: R_Potentiometer, Potentiometer_THT:P120PKY25BR10K, symbol Device:R_Potentiometer
Connections:
- net +3.3V: now also IC1.3 (VOUT), RV1.3
- net +5V: now also IC1.1 (VIN)
- net GND: now also IC1.2 (GND_1), IC1.4 (GND_2), RV1.1
- net Pot_In: now also RV1.2
- no-connect marks 3 -> 1
Other:
- note added: "SWO Pin is not in confirmed location pls check"
- note removed: "SWD Pin is not in confirmed location pls check"
