File: boards/telemetry_GPS/telemetry_GPS_transmitter/can.kicad_sch (KiCad schematic)
At the start: 12 parts, among them J5 54602-908LF, U8 MCP2515-xST, U9 ISO1050DUB

Commit message: Finished Schematic
Parts:
- removed U9: ISO1050DUB, Package_SO:SOP-8_6.62x9.15mm_P2.54mm, symbol Interface_CAN_LIN:ISO1050DUB
- added U8: ISO1042QDWVQ1, ISO1042:DWV0008A-IPC_B, symbol ISO1042:ISO1042QDWVQ1
- renumbered C20 to C21, C21 to C22, C22 to C23, C23 to C24, R9 to R12, R10 to R13, R12 to R14, R11 to R15, U8 to U9
Connections:
- net +3V3: now also U8.1 (VCC1)
- net 5VCAN: now also U8.8 (VCC2)
- net CANH: now also U8.7 (CANH)
- net CANL: now also U8.6 (CANL)
- net CAN_RX: now also U8.3 (RXD)
- net CAN_TX: now also U8.2 (TXD)
- net GND: now also U8.4 (GND1)
- net GNDCAN: now also U8.5 (GND2)
Other:
- moved on the sheet: J5, R15
