File: boards/telemetry_GPS/telemetry_GPS_transmitter/debug.kicad_sch (KiCad schematic)
At the start: 13 parts, among them J2 Conn_02x05_Odd_Even, J3 Conn_01x03, J6 Conn_01x03, SW1 SW_Push, U3 STLINK-V3MODS

Commit message: Finished Schematic
Parts:
- renumbered C14 to C15, J2 to J1, J6 to J2
Connections:
- net SWO: now reaches U3.6 (T_JTDO/T_SWO)
- net SWO: now also J1.5 (Pin_5)
- no-connect marks 21 -> 19
Changed lines of the file:
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@@
 	)
 	(no_connect
-		(at 134.62 118.11)
-	)
-	(no_connect
 		(at 215.9 100.33)
 	)
@@
 	)
 	(no_connect
-		(at 53.34 97.79)
-	)
-	(no_connect
 		(at 215.9 118.11)
 	)
@@
 	(wire
 		(pts
+			(xy 48.26 97.79) (xy 53.34 97.79)
+		)
+		(stroke
+			(width 0)
+			(type default)
+		)
+	)
+	(wire
+		(pts
 			(xy 190.5 66.04) (xy 190.5 68.58)
 		)
@@
 	(wire
 		(pts
+			(xy 129.54 118.11) (xy 134.62 118.11)
+		)
+		(stroke
+			(width 0)
+			(type default)
+		)
+	)
+	(wire
+		(pts
 			(xy 110.49 43.18) (xy 114.3 43.18)
 		)
@@
 		)
 	)
+	(hierarchical_label "SWO"
+		(shape input)
+		(at 129.54 118.11 180)
+		(effects
+			(font
+				(size 1.27 1.27)
+			)
+			(justify right)
+		)
+	)
 	(hierarchical_label "SWCLK"
 		(shape bidirectional)
@@
 		)
 	)
+	(hierarchical_label "SWO"
+		(shape input)
+		(at 48.26 97.79 180)
+		(effects
+			(font
+				(size 1.27 1.27)
+			)
+			(justify right)
+		)
+	)
 	(hierarchical_label "MCU_UART_TX"
 		(shape input)
@@
 		(dnp no)
 		(fields_autoplaced yes)
-		(property "Reference" "C14"
+		(property "Reference" "C15"
 			(at 58.42 140.9699 0)
 			(show_name no)
@@
 			(project "telemetry_GPS_transmitter"
 				(path "/533d07f9-dcec-4fc7-999e-b85b8badcf59/b445cc6d-7b3e-4d39-86ab-3d1fa150ad3f"
-					(reference "C14")
+					(reference "C15")
 					(unit 1)
 				)
@@
 		(dnp no)
 		(fields_autoplaced yes)
-		(property "Reference" "#PWR062"
+		(property "Reference" "#PWR022"
 			(at 48.26 59.69 0)
 			(hide yes)
@@
 			(project "telemetry_GPS_transmitter"
 				(path "/533d07f9-dcec-4fc7-999e-b85b8badcf59/b445cc6d-7b3e-4d39-86ab-3d1fa150ad3f"
-					(reference "#PWR062")
+					(reference "#PWR022")
 					(unit 1)
 				)
@@
 		(dnp no)
 		(fields_autoplaced yes)
-		(property "Reference" "J2"
+		(property "Reference" "J1"
 			(at 59.69 86.36 0)
 			(show_name no)
@@
 			(project "telemetry_GPS_transmitter"
 				(path "/533d07f9-dcec-4fc7-999e-b85b8badcf59/b445cc6d-7b3e-4d39-86ab-3d1fa150ad3f"
-					(reference "J2")
+					(reference "J1")
 					(unit 1)
 				)
@@
 		(dnp no)
 		(fields_autoplaced yes)
-		(property "Reference" "#PWR022"
+		(property "Reference" "#PWR021"
 			(at 46.99 96.52 0)
 			(hide yes)
@@
 			(project "telemetry_GPS_transmitter"
 				(path "/533d07f9-dcec-4fc7-999e-b85b8badcf59/b445cc6d-7b3e-4d39-86ab-3d1fa150ad3f"
-					(reference "#PWR022")
+					(reference "#PWR021")
 					(unit 1)
 				)
@@
 		(dnp no)
 		(fields_autoplaced yes)
-		(property "Reference" "J6"
+		(property "Reference" "J2"
 			(at 62.23 46.9899 0)
 			(show_name no)
@@
 			(project "telemetry_GPS_transmitter"
 				(path "/533d07f9-dcec-4fc7-999e-b85b8badcf59/b445cc6d-7b3e-4d39-86ab-3d1fa150ad3f"
-					(reference "J6")
+					(reference "J2")
 					(unit 1)
 				)
