File: boards/telemetry_GPS/telemetry_GPS_transmitter/debug.kicad_sch (KiCad schematic)
At the start: 14 parts, among them J1 Conn_02x05_Odd_Even, J2 Conn_01x03, J3 Conn_01x03, SW1 SW_Push, U3 STLINK-V3MODS

Commit message: Pushing a finished 2-layer version of the transmitter, will work on 4-layer
Parts:
- JP1, JP2: now not fitted
- U3: now not fitted; now left out of the parts list
- renumbered C14 to C15
Connections:
- net I2C_SCL: now also J3.1 (Pin_1); no longer J3.2 (Pin_2)
- net I2C_SDA: now also J3.2 (Pin_2); no longer J3.1 (Pin_1)
- net MCU_UART_RX: now also J2.1 (Pin_1); no longer J2.2 (Pin_2)
- net MCU_UART_TX: now also J2.2 (Pin_2); no longer J2.1 (Pin_1)

Commit message: Pushing latest fixes
Parts:
- C15: footprint Capacitor_SMD:C_0603_1608Metric_Pad1.08x0.95mm_HandSolder -> Capacitor_SMD:C_0603_1608Metric
- R3, R4, R5: footprint Resistor_SMD:R_0603_1608Metric_Pad0.98x0.95mm_HandSolder -> Resistor_SMD:R_0603_1608Metric
Changed lines of the file:
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@@
 			)
 		)
-		(property "Footprint" "Capacitor_SMD:C_0603_1608Metric_Pad1.08x0.95mm_HandSolder"
+		(property "Footprint" "Capacitor_SMD:C_0603_1608Metric"
 			(at 55.5752 146.05 0)
 			(hide yes)
@@
 			)
 		)
-		(property "Footprint" "Resistor_SMD:R_0603_1608Metric_Pad0.98x0.95mm_HandSolder"
+		(property "Footprint" "Resistor_SMD:R_0603_1608Metric"
 			(at 245.872 64.77 90)
 			(hide yes)
@@
 			)
 		)
-		(property "Footprint" "Resistor_SMD:R_0603_1608Metric_Pad0.98x0.95mm_HandSolder"
+		(property "Footprint" "Resistor_SMD:R_0603_1608Metric"
 			(at 56.642 129.54 90)
 			(hide yes)
@@
 			)
 		)
-		(property "Footprint" "Resistor_SMD:R_0603_1608Metric_Pad0.98x0.95mm_HandSolder"
+		(property "Footprint" "Resistor_SMD:R_0603_1608Metric"
 			(at 228.092 64.77 90)
 			(hide yes)

Commit message: Made a resistor bigger so I can order from ECE Shop
Parts:
- R3: footprint Resistor_SMD:R_0603_1608Metric -> Resistor_SMD:R_0805_2012Metric
Changed lines of the file:
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@@
 			)
 		)
-		(property "Footprint" "Resistor_SMD:R_0603_1608Metric"
+		(property "Footprint" "Resistor_SMD:R_0805_2012Metric"
 			(at 56.642 129.54 90)
 			(hide yes)

Commit message: Pushing finalized design
Connections:
- net MCU_UART_RX: now also J2.2 (Pin_2); no longer J2.1 (Pin_1)
- net MCU_UART_TX: now also J2.1 (Pin_1); no longer J2.2 (Pin_2)
