File: boards/telemetry_GPS/telemetry_GPS_transmitter/gps.kicad_sch (KiCad schematic)
At the start: 5 parts, among them U7 NEO-M8N

Commit message: Finished Schematic
Parts:
- renumbered R7 to R10, R8 to R11, R6 to R9
Changed lines of the file:
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@@
 		(dnp no)
 		(fields_autoplaced yes)
-		(property "Reference" "#PWR043"
+		(property "Reference" "#PWR044"
 			(at 130.81 116.84 0)
 			(hide yes)
@@
 			(project "telemetry_GPS_transmitter"
 				(path "/533d07f9-dcec-4fc7-999e-b85b8badcf59/a7b3cfe0-6bbd-4a95-9258-81caea69e572"
-					(reference "#PWR043")
+					(reference "#PWR044")
 					(unit 1)
 				)
@@
 		(dnp no)
 		(fields_autoplaced yes)
-		(property "Reference" "#PWR044"
+		(property "Reference" "#PWR045"
 			(at 142.24 72.39 0)
 			(hide yes)
@@
 			(project "telemetry_GPS_transmitter"
 				(path "/533d07f9-dcec-4fc7-999e-b85b8badcf59/a7b3cfe0-6bbd-4a95-9258-81caea69e572"
-					(reference "#PWR044")
+					(reference "#PWR045")
 					(unit 1)
 				)
@@
 		(dnp no)
 		(fields_autoplaced yes)
-		(property "Reference" "#PWR047"
+		(property "Reference" "#PWR048"
 			(at 184.15 119.38 0)
 			(hide yes)
@@
 			(project "telemetry_GPS_transmitter"
 				(path "/533d07f9-dcec-4fc7-999e-b85b8badcf59/a7b3cfe0-6bbd-4a95-9258-81caea69e572"
-					(reference "#PWR047")
+					(reference "#PWR048")
 					(unit 1)
 				)
@@
 		(dnp no)
 		(fields_autoplaced yes)
-		(property "Reference" "#PWR046"
+		(property "Reference" "#PWR047"
 			(at 151.13 74.93 0)
 			(hide yes)
@@
 			(project "telemetry_GPS_transmitter"
 				(path "/533d07f9-dcec-4fc7-999e-b85b8badcf59/a7b3cfe0-6bbd-4a95-9258-81caea69e572"
-					(reference "#PWR046")
+					(reference "#PWR047")
 					(unit 1)
 				)
@@
 		(dnp yes)
 		(fields_autoplaced yes)
-		(property "Reference" "R8"
+		(property "Reference" "R11"
 			(at 195.58 105.4099 0)
 			(show_name no)
@@
 			(project "telemetry_GPS_transmitter"
 				(path "/533d07f9-dcec-4fc7-999e-b85b8badcf59/a7b3cfe0-6bbd-4a95-9258-81caea69e572"
-					(reference "R8")
+					(reference "R11")
 					(unit 1)
 				)
@@
 		(dnp yes)
 		(fields_autoplaced yes)
-		(property "Reference" "R6"
+		(property "Reference" "R9"
 			(at 177.8 105.4099 0)
 			(show_name no)
@@
 			(project "telemetry_GPS_transmitter"
 				(path "/533d07f9-dcec-4fc7-999e-b85b8badcf59/a7b3cfe0-6bbd-4a95-9258-81caea69e572"
-					(reference "R6")
+					(reference "R9")
 					(unit 1)
 				)
@@
 		(dnp no)
 		(fields_autoplaced yes)
-		(property "Reference" "#PWR045"
+		(property "Reference" "#PWR046"
 			(at 147.32 132.08 0)
 			(hide yes)
@@
 			(project "telemetry_GPS_transmitter"
 				(path "/533d07f9-dcec-4fc7-999e-b85b8badcf59/a7b3cfe0-6bbd-4a95-9258-81caea69e572"
-					(reference "#PWR045")
+					(reference "#PWR046")
 					(unit 1)
 				)
@@
 		(dnp no)
 		(fields_autoplaced yes)
-		(property "Reference" "R7"
+		(property "Reference" "R10"
 			(at 184.15 92.71 90)
 			(show_name no)
@@
 			(project "telemetry_GPS_transmitter"
 				(path "/533d07f9-dcec-4fc7-999e-b85b8badcf59/a7b3cfe0-6bbd-4a95-9258-81caea69e572"
-					(reference "R7")
-					(unit 1)
-				)
+					(reference "R10")
+					(unit 1)
+				)
