File: boards/telemetry_GPS/telemetry_GPS_transmitter/ldo.kicad_sch (KiCad schematic)
At the start: 5 parts, among them U2 TLV75509PDBV

Commit message: Finished Schematic
Parts:
- C13: renamed from C12; value 0.1uF -> 1uF
- C14: renamed from C13; value 0.1uF -> 1uF
Changed lines of the file:
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@@
 		(dnp no)
 		(fields_autoplaced yes)
-		(property "Reference" "C12"
+		(property "Reference" "C13"
 			(at 80.01 77.4699 0)
 			(show_name no)
@@
 			)
 		)
-		(property "Value" "0.1uF"
+		(property "Value" "1uF"
 			(at 80.01 80.0099 0)
 			(show_name no)
@@
 			(project "telemetry_GPS_transmitter"
 				(path "/533d07f9-dcec-4fc7-999e-b85b8badcf59/8a3a1144-1204-45bc-8a8c-54e20062ae57"
-					(reference "C12")
+					(reference "C13")
 					(unit 1)
 				)
@@
 		(dnp no)
 		(fields_autoplaced yes)
-		(property "Reference" "#PWR019"
+		(property "Reference" "#PWR020"
 			(at 121.92 91.44 0)
 			(hide yes)
@@
 			(project "telemetry_GPS_transmitter"
 				(path "/533d07f9-dcec-4fc7-999e-b85b8badcf59/8a3a1144-1204-45bc-8a8c-54e20062ae57"
-					(reference "#PWR019")
+					(reference "#PWR020")
 					(unit 1)
 				)
@@
 		(dnp no)
 		(fields_autoplaced yes)
-		(property "Reference" "#PWR016"
+		(property "Reference" "#PWR017"
 			(at 88.9 91.44 0)
 			(hide yes)
@@
 			(project "telemetry_GPS_transmitter"
 				(path "/533d07f9-dcec-4fc7-999e-b85b8badcf59/8a3a1144-1204-45bc-8a8c-54e20062ae57"
-					(reference "#PWR016")
+					(reference "#PWR017")
 					(unit 1)
 				)
@@
 		(dnp no)
 		(fields_autoplaced yes)
-		(property "Reference" "#PWR015"
+		(property "Reference" "#PWR016"
 			(at 69.85 68.58 0)
 			(hide yes)
@@
 			(project "telemetry_GPS_transmitter"
 				(path "/533d07f9-dcec-4fc7-999e-b85b8badcf59/8a3a1144-1204-45bc-8a8c-54e20062ae57"
-					(reference "#PWR015")
+					(reference "#PWR016")
 					(unit 1)
 				)
@@
 		(dnp no)
 		(fields_autoplaced yes)
-		(property "Reference" "#PWR018"
+		(property "Reference" "#PWR019"
 			(at 121.92 67.31 0)
 			(hide yes)
@@
 			(project "telemetry_GPS_transmitter"
 				(path "/533d07f9-dcec-4fc7-999e-b85b8badcf59/8a3a1144-1204-45bc-8a8c-54e20062ae57"
-					(reference "#PWR018")
+					(reference "#PWR019")
 					(unit 1)
 				)
@@
 		(dnp no)
 		(fields_autoplaced yes)
-		(property "Reference" "C13"
+		(property "Reference" "C14"
 			(at 104.14 77.4699 0)
 			(show_name no)
@@
 			)
 		)
-		(property "Value" "0.1uF"
+		(property "Value" "1uF"
 			(at 104.14 80.0099 0)
 			(show_name no)
@@
 			(project "telemetry_GPS_transmitter"
 				(path "/533d07f9-dcec-4fc7-999e-b85b8badcf59/8a3a1144-1204-45bc-8a8c-54e20062ae57"
-					(reference "C13")
+					(reference "C14")
 					(unit 1)
 				)
@@
 		(dnp no)
 		(fields_autoplaced yes)
-		(property "Reference" "#PWR017"
+		(property "Reference" "#PWR018"
 			(at 105.41 68.58 0)
 			(hide yes)
@@
 			(project "telemetry_GPS_transmitter"
 				(path "/533d07f9-dcec-4fc7-999e-b85b8badcf59/8a3a1144-1204-45bc-8a8c-54e20062ae57"
-					(reference "#PWR017")
-					(unit 1)
-				)
+					(reference "#PWR018")
+					(unit 1)
+				)
