File: boards/telemetry_GPS/telemetry_GPS_transmitter/stm32.kicad_sch (KiCad schematic)
At the start: 16 parts, among them U1 STM32WL55CCUx

Commit message: Finished Schematic
Parts:
- removed NT1: NetTie_2, NetTie:NetTie-2_SMD_Pad0.5mm, symbol Device:NetTie_2
- added C1: 10pF, Capacitor_SMD:C_0603_1608Metric_Pad1.08x0.95mm_HandSolder, symbol Device:C
- renumbered C9 to C10, C10 to C11, C11 to C12, C1 to C2, C2 to C3, C3 to C4, C4 to C5, C5 to C6, C6 to C7, C7 to C8, C8 to C9
Connections:
- net VSS_SMPS is gone; now on net GND: C3.2, C5.2, U1.48 (VSSSMPS)
- net OSC_IN: now also C1.1; no longer XTAL1.3
- net OSC_OUT: now also XTAL1.3; no longer XTAL1.1
- net SPI1_SCK: now also U1.13 (PA5); no longer U1.1 (PB3)
- new net: C1.2, XTAL1.1
- new net SWO: U1.1 (PB3)
- no-connect marks 10 -> 9
Other:
- note added: "Refer to VSSSMPS"
