File: boards/telemetry_GPS/telemetry_GPS_transmitter/telemetry_GPS_transmitter.kicad_sch (KiCad schematic)
At the start: 0 parts

Commit message: Finished Schematic
Other:
- sheet Debug ports: added SWO; removed none
- sheet STM32 ports: added SWO; removed none
Changed lines of the file:
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@@
+	(wire
+		(pts
+			(xy 148.59 88.9) (xy 172.72 88.9)
+		)
+		(stroke
+			(width 0)
+			(type default)
+		)
+	)
 	(wire
 		(pts
@@
 	(wire
 		(pts
-			(xy 148.59 88.9) (xy 172.72 88.9)
+			(xy 148.59 91.44) (xy 172.72 91.44)
 		)
 		(stroke
@@
 	(wire
 		(pts
-			(xy 148.59 91.44) (xy 172.72 91.44)
+			(xy 148.59 93.98) (xy 172.72 93.98)
 		)
 		(stroke
@@
 			)
 		)
-		(pin "SWDIO" bidirectional
+		(pin "SWDIO" output
 			(at 148.59 86.36 0)
 			(effects
@@
 		)
 		(pin "USART2_RX" input
-			(at 148.59 88.9 0)
+			(at 148.59 91.44 0)
 			(effects
 				(font
@@
 		)
 		(pin "USART2_TX" input
-			(at 148.59 91.44 0)
+			(at 148.59 93.98 0)
 			(effects
 				(font
@@
 				)
 				(justify left)
+			)
+		)
+		(pin "SWO" output
+			(at 148.59 88.9 0)
+			(effects
+				(font
+					(size 1.27 1.27)
+				)
+				(justify right)
 			)
 		)
@@
 	(sheet
 		(at 172.72 67.31)
-		(size 19.05 28.194)
+		(size 19.05 31.496)
 		(exclude_from_sim no)
 		(in_bom yes)
@@
 		)
 		(property "Sheetfile" "debug.kicad_sch"
-			(at 172.72 96.0886 0)
+			(at 172.72 99.3906 0)
 			(show_name no)
 			(do_not_autoplace no)
@@
 		)
 		(pin "MCU_UART_RX" output
-			(at 172.72 88.9 180)
+			(at 172.72 91.44 180)
 			(effects
 				(font
@@
 		)
 		(pin "MCU_UART_TX" input
-			(at 172.72 91.44 180)
+			(at 172.72 93.98 180)
 			(effects
 				(font
@@
 			(effects
 				(font
+					(size 1.27 1.27)
+				)
+				(justify left)
+			)
+		)
+		(pin "SWO" input
+			(at 172.72 88.9 180)
+			(effects
+				(font

Commit message: Pushing some antenna routing stuff
Parts:
- added H1, H2, H3, H4: MountingHole, MountingHole:MountingHole_4.3mm_M4, symbol Mechanical:MountingHole
