File: boards/telemetry_GPS/telemetry_GPS_transmitter/telemetry_GPS_transmitter.kicad_sch (KiCad schematic)
At the start: 4 parts

Commit message: Pushing a finished 2-layer version of the transmitter, will work on 4-layer
Changed lines of the file:
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@@
-		)
-	)
-	(symbol
-		(lib_id "EVCLogo:LOGO")
-		(at 243.84 99.06 0)
-		(unit 1)
-		(body_style 1)
-		(exclude_from_sim no)
-		(in_bom yes)
-		(on_board yes)
-		(in_pos_files yes)
-		(dnp no)
-		(fields_autoplaced yes)
-		(property "Reference" "#G1"
-			(at 243.84 55.723 0)
-			(hide yes)
-			(show_name no)
-			(do_not_autoplace no)
-			(effects
-				(font
-					(size 1.27 1.27)
-				)
-			)
-		)
-		(property "Value" "LOGO"
-			(at 243.84 142.397 0)
-			(hide yes)
-			(show_name no)
-			(do_not_autoplace no)
-			(effects
-				(font
-					(size 1.27 1.27)
-				)
-			)
-		)
-		(property "Footprint" "EVC Logo:EVC_LOGO"
-			(at 243.84 99.06 0)
-			(hide yes)
-			(show_name no)
-			(do_not_autoplace no)
-			(effects
-				(font
-					(size 1.27 1.27)
-				)
-			)
-		)
-		(property "Datasheet" ""
-			(at 243.84 99.06 0)
-			(hide yes)
-			(show_name no)
-			(do_not_autoplace no)
-			(effects
-				(font
-					(size 1.27 1.27)
-				)
-			)
-		)
-		(property "Description" ""
-			(at 243.84 99.06 0)
-			(hide yes)
-			(show_name no)
-			(do_not_autoplace no)
-			(effects
-				(font
-					(size 1.27 1.27)
-				)
-			)
-		)
-		(instances
-			(project "telemetry_GPS_transmitter"
-				(path "/533d07f9-dcec-4fc7-999e-b85b8badcf59"
-					(reference "#G1")
-					(unit 1)
-				)
-			)
 		)
 	)
