File: boards/telemetry_GPS/telemetry_GPS_transmitter/rf-backup.kicad_sch (KiCad schematic)
At the start: 11 parts

Commit message: Pushing a finished 2-layer version of the transmitter, will work on 4-layer
Parts:
- renumbered C24 to C25, C25 to C26, C26 to C27, C27 to C28, C28 to C29, C29 to C30, C30 to C31
Changed lines of the file:
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@@
 		(dnp no)
 		(fields_autoplaced yes)
-		(property "Reference" "C26"
+		(property "Reference" "C27"
 			(at 106.68 83.8199 0)
 			(show_name no)
@@
 			(project "telemetry_GPS_transmitter"
 				(path "/533d07f9-dcec-4fc7-999e-b85b8badcf59/e71ddfbd-55e3-49a6-8efb-57936fc9e5b8"
-					(reference "C26")
+					(reference "C27")
 					(unit 1)
 				)
@@
 		(dnp no)
 		(fields_autoplaced yes)
-		(property "Reference" "C28"
+		(property "Reference" "C29"
 			(at 124.46 83.8199 0)
 			(show_name no)
@@
 			(project "telemetry_GPS_transmitter"
 				(path "/533d07f9-dcec-4fc7-999e-b85b8badcf59/e71ddfbd-55e3-49a6-8efb-57936fc9e5b8"
-					(reference "C28")
+					(reference "C29")
 					(unit 1)
 				)
@@
 		(dnp no)
 		(fields_autoplaced yes)
-		(property "Reference" "#PWR061"
+		(property "Reference" "#PWR058"
 			(at 78.74 72.39 0)
 			(hide yes)
@@
 			(project "telemetry_GPS_transmitter"
 				(path "/533d07f9-dcec-4fc7-999e-b85b8badcf59/e71ddfbd-55e3-49a6-8efb-57936fc9e5b8"
-					(reference "#PWR061")
+					(reference "#PWR058")
 					(unit 1)
 				)
@@
 		(dnp no)
 		(fields_autoplaced yes)
-		(property "Reference" "#PWR062"
+		(property "Reference" "#PWR059"
 			(at 111.76 97.79 0)
 			(hide yes)
@@
 			(project "telemetry_GPS_transmitter"
 				(path "/533d07f9-dcec-4fc7-999e-b85b8badcf59/e71ddfbd-55e3-49a6-8efb-57936fc9e5b8"
-					(reference "#PWR062")
+					(reference "#PWR059")
 					(unit 1)
 				)
@@
 		(dnp no)
 		(fields_autoplaced yes)
-		(property "Reference" "#PWR063"
+		(property "Reference" "#PWR060"
 			(at 149.86 97.79 0)
 			(hide yes)
@@
 			(project "telemetry_GPS_transmitter"
 				(path "/533d07f9-dcec-4fc7-999e-b85b8badcf59/e71ddfbd-55e3-49a6-8efb-57936fc9e5b8"
-					(reference "#PWR063")
+					(reference "#PWR060")
 					(unit 1)
 				)
@@
 		(dnp no)
 		(fields_autoplaced yes)
-		(property "Reference" "C27"
+		(property "Reference" "C28"
 			(at 114.3 62.23 90)
 			(show_name no)
@@
 			(project "telemetry_GPS_transmitter"
 				(path "/533d07f9-dcec-4fc7-999e-b85b8badcf59/e71ddfbd-55e3-49a6-8efb-57936fc9e5b8"
-					(reference "C27")
+					(reference "C28")
 					(unit 1)
 				)
@@
 		(dnp no)
 		(fields_autoplaced yes)
-		(property "Reference" "C29"
+		(property "Reference" "C30"
 			(at 128.27 71.12 90)
 			(show_name no)
@@
 			(project "telemetry_GPS_transmitter"
 				(path "/533d07f9-dcec-4fc7-999e-b85b8badcf59/e71ddfbd-55e3-49a6-8efb-57936fc9e5b8"
-					(reference "C29")
+					(reference "C30")
 					(unit 1)
 				)
@@
 		(dnp no)
 		(fields_autoplaced yes)
-		(property "Reference" "C24"
+		(property "Reference" "C25"
 			(at 76.2 60.9599 0)
 			(show_name no)
@@
 			(project "telemetry_GPS_transmitter"
 				(path "/533d07f9-dcec-4fc7-999e-b85b8badcf59/e71ddfbd-55e3-49a6-8efb-57936fc9e5b8"
-					(reference "C24")
+					(reference "C25")
 					(unit 1)
 				)
@@
 		(dnp no)
 		(fields_autoplaced yes)
-		(property "Reference" "C25"
+		(property "Reference" "C26"
 			(at 88.9 60.9599 0)
 			(show_name no)
@@
 			(project "telemetry_GPS_transmitter"
 				(path "/533d07f9-dcec-4fc7-999e-b85b8badcf59/e71ddfbd-55e3-49a6-8efb-57936fc9e5b8"
-					(reference "C25")
+					(reference "C26")
 					(unit 1)
 				)
@@
 		(dnp no)
 		(fields_autoplaced yes)
-		(property "Reference" "C30"
+		(property "Reference" "C31"
 			(at 153.67 83.8199 0)
 			(show_name no)
@@
 			(project "telemetry_GPS_transmitter"
 				(path "/533d07f9-dcec-4fc7-999e-b85b8badcf59/e71ddfbd-55e3-49a6-8efb-57936fc9e5b8"
-					(reference "C30")
-					(unit 1)
-				)
+					(reference "C31")
+					(unit 1)
+				)
