File: boards/DashboardV2.0/DashboardV2.0.kicad_sch (KiCad schematic)
At the start: 0 parts

Commit message: Made a sheet (LCD) for schematic
Testing out if we can make hierarchical subsheets.
Other:
- added sheet LCD (LCD_sch.kicad_sch)
Changed lines of the file:
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@@
 	(generator_version "10.0")
 	(paper "A4")
+	(sheet
+		(at 160.02 40.64)
+		(size 63.5 50.8)
+		(exclude_from_sim no)
+		(in_bom yes)
+		(on_board yes)
+		(dnp no)
+		(fields_autoplaced yes)
+		(stroke
+			(width 0.1524)
+			(type solid)
+		)
+		(fill
+			(color 0 0 0 0)
+		)
+		(property "Sheetname" "LCD"
+			(at 160.02 39.9284 0)
+			(show_name no)
+			(do_not_autoplace no)
+			(effects
+				(font
+					(size 1.27 1.27)
+				)
+				(justify left bottom)
+			)
+		)
+		(property "Sheetfile" "LCD_sch.kicad_sch"
+			(at 160.02 92.0246 0)
+			(show_name no)
+			(do_not_autoplace no)
+			(effects
+				(font
+					(size 1.27 1.27)
+				)
+				(justify left top)
+			)
+		)
+		(instances
+			(project "DashboardV2.0"
+				(path "/11d8d7d9-6006-4d5e-8823-06d4aec43d5d"
+					(page "2")
+				)
+			)
+		)
+	)
 	(sheet_instances
 		(path "/"
