File: boards/DashboardV2.0/EVC Dashboard V2/flashmemory.kicad_sch (KiCad schematic)
At the start: 0 parts

Commit message: Added MCU, UI, and Flash
Added more connections to the MCU, added in switches for UI and the flash memory. Will continue finishing MCU connections, need to add can connector and LCD connections.
Parts:
- added 111: MT25QL128ABA1EW9-0SIT, dashboardgen2:SON127P800X600X80-9N-D, symbol dashBoardGen2:MT25QL128ABA1EW9-0SIT
- added C35: .1uF, Capacitor_SMD:C_0603_1608Metric, symbol Device:C
- added R10: 10K, Resistor_SMD:R_0402_1005Metric, symbol Device:R
Connections:
- new net +3V3: 111.8 (V_CC), C35.1, R10.1
- new net GND: 111.4 (V_SS), 111.9 (GND), C35.2
- new net QSPI_BK1_IO0: 111.5 (DQ0)
- new net QSPI_BK1_IO1: 111.2 (DQ1)
- new net QSPI_BK1_IO2: 111.3 (W#/DQ2)
- new net QSPI_BK1_IO3: 111.7 (DQ3/HOLD#)
- new net QSPI_BK1_NCS: 111.1 (S#), R10.2
- new net QSPI_CLK: 111.6 (C)
