File: boards/DashboardV2.0/EVC Dashboard V2/userinputs.kicad_sch (KiCad schematic)
At the start: 0 parts

Commit message: Added MCU, UI, and Flash
Added more connections to the MCU, added in switches for UI and the flash memory. Will continue finishing MCU connections, need to add can connector and LCD connections.
Parts:
- added C73, C74, C76, C77, C79, C80, C81, C82, C83, C84: .1uF, Capacitor_SMD:C_0603_1608Metric, symbol Device:C
- added R19, R20, R26, R27, R33, R34, R39, R40, R45, R46: 100R, Resistor_SMD:R_0603_1608Metric, symbol Device:R
- added R21, R22, R29, R30, R35, R36, R41, R42, R47, R48: 220K, Resistor_SMD:R_0603_1608Metric, symbol Device:R
- added R24, R25, R31, R32, R37, R38, R43, R44, R49, R50: 330R, Resistor_SMD:R_0603_1608Metric, symbol Device:R
- added SW10, SW11, SW2, SW3, SW4, SW5, SW6, SW7, SW8, SW9: SW_Push, dashboardgen2:5GSH920, symbol Switch:SW_Push
Connections:
- new net: C76.1, R26.1
- new net: C76.2, R29.2, R31.2, SW3.2
- new net: C79.2, R35.2, R37.2, SW4.2
- new net: C81.1, R39.1
- new net: C77.2, R30.1, R32.2, SW6.2
- new net: C82.1, R40.1
- new net: C84.2, R48.2, R50.2, SW11.2
- new net: C77.1, R27.1
- new net: C80.2, R36.2, R38.2, SW7.2
- new net: C84.1, R46.1
- new net: C73.2, R21.2, R24.2, SW2.2
- new net: C81.2, R41.2, R43.2, SW8.2
- new net: C74.1, R20.1
- new net: C74.2, R22.2, R25.2, SW5.2
- new net: C83.2, R47.2, R49.2, SW10.2
- new net: C83.1, R45.1
- new net: C82.2, R42.2, R44.2, SW9.2
- new net: C79.1, R33.1
- new net: C73.1, R19.1
- new net: C80.1, R34.1
- new net +3V3: R19.2, R20.2, R26.2, R27.2, R33.2, R34.2, R39.2, R40.2, R45.2, R46.2, SW10.1, SW11.1, SW2.1, SW3.1, SW4.1, SW5.1, SW6.1, SW7.1, SW8.1, SW9.1
- new net GND: R21.1, R22.1, R29.1, R30.2, R35.1, R36.1, R41.1, R42.1, R47.1, R48.1
- new net SW_0: R24.1
- new net SW_1: R31.1
- new net SW_2: R37.1
- new net SW_3: R43.1
- new net SW_4: R49.1
- new net SW_5: R25.1
- new net SW_6: R32.1
- new net SW_7: R38.1
- new net SW_8: R44.1
- new net SW_9: R50.1

Commit message: Encoders
Parts:
- added C75, C88: .1uF, Capacitor_SMD:C_0603_1608Metric, symbol Device:C
- added C78, C89, C90, C91: .01uF, Capacitor_SMD:C_0603_1608Metric, symbol Device:C
- added R23, R51: 100R, Resistor_SMD:R_0603_1608Metric, symbol Device:R
- added R28, R52: 220K, Resistor_SMD:R_0603_1608Metric, symbol Device:R
- added R53, R58: 330R, Resistor_SMD:R_0603_1608Metric, symbol Device:R
- added R54, R55, R56, R57, R59, R60, R61, R62: 10k, Resistor_SMD:R_0603_1608Metric, symbol Device:R
- added SW12, SW13: PEC12-4222F, dashboardgen2:PEC12R-4222F-S0024, symbol dashBoardGen2:PEC12R-4222F-S0024
Connections:
- net +3V3: now also R23.2, R51.2, R54.1, R56.1, R59.1, R60.1, SW12.1, SW13.1
- net GND: now also C78.2, C89.2, C90.2, C91.2, R28.1, R52.1, SW12.4 (C), SW12.6 (BODY), SW12.7 (BODY), SW13.4 (C), SW13.6 (BODY), SW13.7 (BODY)
- new net: C75.2, R28.2, R58.2, SW13.2
- new net: R59.2, R61.1, SW13.3 (A)
- new net: R60.2, R62.1, SW13.5 (B)
- new net: C88.2, R52.2, R53.2, SW12.2
- new net: C75.1, R23.1
- new net: R54.2, R55.1, SW12.3 (A)
- new net: R56.2, R57.1, SW12.5 (B)
- new net: C88.1, R51.1
- new net ENC1A: C89.1, R55.2
- new net ENC1B: C90.1, R57.2
- new net ENC2A: C78.1, R61.2
- new net ENC2B: C91.1, R62.2
- new net SW_10: R53.1
- new net SW_11: R58.1
Other:
- note added: "Encoders"
- note added: "Switches"
- moved on the sheet: C73, C74, C76, C77, C79, C80, C81, C82, C83, C84, R19, R20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
