File: boards/DashboardV2.0/EVC Dashboard V2/EVC Dashboard V2.kicad_sch (KiCad schematic)
At the start: 0 parts

Commit message: Added overvoltage subsheet
Other:
- added sheet Overvoltage Protection (overvoltage.kicad_sch)
Changed lines of the file:
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@@
+	)
+	(sheet
+		(at 105.41 167.64)
+		(size 63.5 25.4)
+		(exclude_from_sim no)
+		(in_bom yes)
+		(on_board yes)
+		(dnp no)
+		(fields_autoplaced yes)
+		(stroke
+			(width 0.1524)
+			(type solid)
+		)
+		(fill
+			(color 0 0 0 0)
+		)
+		(property "Sheetname" "Overvoltage Protection"
+			(at 105.41 166.9284 0)
+			(show_name no)
+			(do_not_autoplace no)
+			(effects
+				(font
+					(size 1.27 1.27)
+				)
+				(justify left bottom)
+			)
+		)
+		(property "Sheetfile" "overvoltage.kicad_sch"
+			(at 105.41 193.6246 0)
+			(show_name no)
+			(do_not_autoplace no)
+			(effects
+				(font
+					(size 1.27 1.27)
+				)
+				(justify left top)
+			)
+		)
+		(instances
+			(project "EVC Dashboard V2"
+				(path "/ede78d5d-1d5c-4e8d-a13e-c039265851a9"
+					(page "9")
+				)
+			)
+		)
 	)
 	(sheet

Commit message: Added oscillators and ferrite bead to MCU
Added the remaining MCU parts, will add NC and LED_CAN to finish MCU connections
Parts:
- added H1, H2, H3, H4, H5, H6: MountingHole, MountingHole:MountingHole_3.2mm_M3, symbol Mechanical:MountingHole
