File: boards/DashboardV2.0/EVC Dashboard V2/MCU.kicad_sch (KiCad schematic)
At the start: 0 parts

Commit message: Added Dashboard MCU Connections
Started wiring MCU connections that are unrelated to display, after deciding on display, will finish wiring MCU
Parts:
- added R1, R3: R, Package_QFP:LQFP-144_20x20mm_P0.5mm, symbol Device:R
- added R2, R4: R, symbol Device:R
- added U1: STM32H750ZBTx, Package_QFP:LQFP-144_20x20mm_P0.5mm, symbol MCU_ST_STM32H7:STM32H750ZBTx
Connections:
- new net: R1.2, R2.1, U1.138 (BOOT0)
- new net: R3.2, R4.1, U1.143 (PDR_ON)
- new net +3.3V: R1.1, R3.1, U1.108 (VDD), U1.121 (VDD), U1.131 (VDD), U1.144 (VDD), U1.17 (VDD), U1.30 (VDD), U1.39 (VDD), U1.52 (VDD), U1.6 (VBAT), U1.62 (VDD), U1.72 (VDD), U1.84 (VDD)
- new net A0: U1.10 (PF0)
- new net A1: U1.11 (PF1)
- new net A2: U1.12 (PF2)
- new net A3: U1.13 (PF3)
- new net A4: U1.14 (PF4)
- new net A5: U1.15 (PF5)
- new net CAN_RX: U1.103 (PA11)
- new net CAN_TX: U1.104 (PA12)
- new net GND: U1.107 (VSS), U1.120 (VSS), U1.130 (VSS), U1.16 (VSS), U1.31 (VSSA), U1.38 (VSS), U1.51 (VSS), U1.61 (VSS), U1.83 (VSS), U1.94 (VSS)
- new net I2C1_SCL: U1.139 (PB8)
- new net I2C1_SDA: U1.137 (PB7)
- new net I2C3_SCL: U1.100 (PA8)
- new net NRST: U1.25 (NRST)
- new net QSPI_CLK: U1.48 (PB2)
- new net QUADSPI_BK1_IO0: U1.80 (PD11)
- new net QUADSPI_BK1_IO1: U1.81 (PD12)
- new net QUADSPI_BK1_IO2: U1.1 (PE2)
- new net QUADSPI_BK1_IO3: U1.82 (PD13)
- new net QUADSPI_BK1_NCS: U1.136 (PB6)
- new net SWCLK: U1.109 (PA14)
- new net SWDIO: U1.105 (PA13)
- new net SWO: U1.133 (PB3)
- new net VREF: U1.32 (VREF+)

Commit message: Added MCU, UI, and Flash
Added more connections to the MCU, added in switches for UI and the flash memory. Will continue finishing MCU connections, need to add can connector and LCD connections.
Parts:
- added C10, C11, C12, C13, C14, C15, C16, C17, C18, C19, C20, C26, C27, C34: 100n, Capacitor_SMD:C_0402_1005Metric, symbol Device:C
- added C8, C9: 2.2u, Capacitor_SMD:C_0603_1608Metric, symbol Device:C
- added D3, D4, D5, D6, D7, D8, D9: LED, LED_SMD:LED_0603_1608Metric, symbol Device:LED
- added J8: Conn_02x05_Odd_Even, Connector_PinSocket_2.54mm:PinSocket_2x05_P2.54mm_Vertical, symbol Connector_Generic:Conn_02x05_Odd_Even
- added R69, R70, R71, R72, R73, R74, R75: 300, Resistor_SMD:R_0805_2012Metric, symbol Device:R
Connections:
- net GND: now also R2.2, R4.2, C10.2, C11.2, C12.2, C13.2, C14.2, C15.2, C16.2, C17.2, C18.2, C19.2, C20.2, C26.2, C27.2, C34.2, C8.1, C9.1, J8.10 (Pin_10), J8.9 (Pin_9), R69.1, R70.1, R71.1, R72.1, R73.1, R74.1, R75.1
- net at U1.106 (VCAP): now also C9.2
- net LED2: now reaches U1.111 (PC10)
- net LED2: now also D4.2 (A), J8.2 (Pin_2)
- net LED3: now reaches U1.112 (PC11)
- net LED3: now also D5.2 (A), J8.3 (Pin_3)
- net SW_0: now reaches U1.26 (PC0)
- net SW_1: now reaches U1.27 (PC1)
- net SW_2: now reaches U1.28 (PC2_C)
- net SW_3: now reaches U1.29 (PC3_C)
- net DSX: now reaches U1.35 (PA1)
- net RESX: now reaches U1.36 (PA2)
- net TE: now reaches U1.37 (PA3)
- net CSX: now reaches U1.40 (PA4)
- net SCL: now reaches U1.41 (PA5)
- net MISO: now reaches U1.42 (PA6)
- net MOSI: now reaches U1.43 (PA7)
- net SW_8: now reaches U1.46 (PB0)
- net SW_9: now reaches U1.47 (PB1)
- net LED1: now reaches U1.70 (PB11)
- net LED1: now also D3.2 (A), J8.1 (Pin_1)
- net at U1.71 (VCAP): now also C8.2
- net SW_4: now reaches U1.96 (PC6)
- net SW_5: now reaches U1.97 (PC7)
- net SW_6: now reaches U1.98 (PC8)
- net SW_7: now reaches U1.99 (PC9)
- net A0: no longer names the net of U1.10 (PF0)
- net A1: no longer names the net of U1.11 (PF1)
- net A2: no longer names the net of U1.12 (PF2)
- net A3: no longer names the net of U1.13 (PF3)
- net A4: no longer names the net of U1.14 (PF4)
- net A5: no longer names the net of U1.15 (PF5)
- net QUADSPI_BK1_IO0 renamed QSPI_BK1_IO0
- net QUADSPI_BK1_IO1 renamed QSPI_BK1_IO1
- net QUADSPI_BK1_IO2 renamed QSPI_BK1_IO2
- net QUADSPI_BK1_IO3 renamed QSPI_BK1_IO3
- net QUADSPI_BK1_NCS renamed QSPI_BK1_NCS
- new net: D7.1 (K), R73.2
- new net: D4.1 (K), R70.2
- new net: D6.1 (K), R72.2
- new net: D9.1 (K), R75.2
- new net: D5.1 (K), R71.2
- new net: D3.1 (K), R69.2
- new net: D8.1 (K), R74.2
- new net +3V3: C10.1, C11.1, C12.1, C13.1, C14.1, C15.1, C16.1, C17.1, C18.1, C19.1, C20.1, C26.1, C27.1, C34.1, J8.8 (Pin_8)
- new net LED4: D6.2 (A), J8.4 (Pin_4)
- new net LED5: D7.2 (A), J8.5 (Pin_5)
- new net LED6: D8.2 (A), J8.6 (Pin_6)
- new net LED7: D9.2 (A), J8.7 (Pin_7)
Other:
- note added: "Decoupling Caps"
- moved on the sheet: R1, R2, R3, R4, U1

Commit message: Added oscillators and ferrite bead to MCU
Added the remaining MCU parts, will add NC and LED_CAN to finish MCU connections
Parts:
- added C21, C7: 8pF, Capacitor_SMD:C_0402_1005Metric, symbol Device:C
- added C22, C23: 12.5pF, Capacitor_SMD:C_0402_1005Metric, symbol Device:C
- added FB1: FerriteBead, Inductor_SMD:L_0603_1608Metric, symbol Device:FerriteBead
- added R13: 0, Resistor_SMD:R_0603_1608Metric, symbol Device:R
- added X1: 8Mhz, dashboardgen2:NX3225GD8MHZSTDCRA3, symbol Crystals & Oscillators:NX3225GD-8MHZ-STD-CRA-3
- added X2: 32K, dashboardgen2:NX3215SA32768KSTDMUA8, symbol dashBoardGen2:NX3215SA-32.768K-STD-MUA-8
Connections:
- net +3.3V: now also U1.95 (VDD33_USB)
- net +3V3: now also FB1.2
- net GND: now also C22.1, C23.1
- net VREF: now also R13.1
- net at U1.23 (PH0): now also C7.2, X1.2
- net at U1.24 (PH1): now also C21.2, X1.1
- net at U1.33 (VDDA): now also FB1.1, R13.2
- net at U1.8 (PC14): now also C22.2, X2.1
- net at U1.9 (PC15): now also C23.2, X2.2 (CRYSTAL_2)
- new net: C21.1, C7.1

Commit message: Added MCU Labels
Finished adding labels for LEDs and CAN indicator LED
Connections:
- net LED1: now also U1.134 (PB4); no longer U1.70 (PB11)
- net LED2: now also U1.135 (PB5); no longer U1.111 (PC10)
- net LED3: now also U1.140 (PB9), U1.69 (PB10); no longer U1.112 (PC11)
- net LED4: now also U1.70 (PB11)
- net LED5: now also U1.73 (PB12)
- net LED6: now also U1.74 (PB13)
- net LED7: now also U1.75 (PB14)
- net LED_CAN: now reaches U1.76 (PB15)
Changed lines of the file:
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@@
+		)
+	)
+	(label "LED3"
+		(at 222.25 130.81 0)
+		(effects
+			(font
+				(size 1.27 1.27)
+			)
+			(justify left bottom)
 		)
 	)
@@
 		)
 	)
+	(label "LED4"
+		(at 222.25 133.35 0)
+		(effects
+			(font
+				(size 1.27 1.27)
+			)
+			(justify left bottom)
+		)
+	)
+	(label "LED6"
+		(at 222.25 138.43 0)
+		(effects
+			(font
+				(size 1.27 1.27)
+			)
+			(justify left bottom)
+		)
+	)
 	(label "LED1"
 		(at 64.77 107.315 180)
@@
 	)
 	(label "LED1"
+		(at 222.25 115.57 0)
+		(effects
+			(font
+				(size 1.27 1.27)
+			)
+			(justify left bottom)
+		)
+	)
+	(label "LED5"
+		(at 222.25 135.89 0)
+		(effects
+			(font
+				(size 1.27 1.27)
+			)
+			(justify left bottom)
+		)
+	)
+	(label "LED2"
+		(at 222.25 118.11 0)
+		(effects
+			(font
+				(size 1.27 1.27)
+			)
+			(justify left bottom)
+		)
+	)
+	(label "LED1"
 		(at 64.135 139.065 180)
 		(effects
@@
 			)
 			(justify right bottom)
+		)
+	)
+	(label "LED7"
+		(at 222.25 140.97 0)
+		(effects
+			(font
+				(size 1.27 1.27)
+			)
+			(justify left bottom)
 		)
 	)
@@
 		)
 	)
-	(global_label "LED1"
-		(shape input)
-		(at 222.25 133.35 0)
-		(fields_autoplaced yes)
-		(effects
-			(font
-				(size 1.27 1.27)
-			)
-			(justify left)
-		)
-		(property "Intersheetrefs" "${INTERSHEET_REFS}"
-			(at 229.8918 133.35 0)
+	(global_label "LED3"
+		(shape input)
+		(at 228.6 128.27 0)
+		(fields_autoplaced yes)
+		(effects
+			(font
+				(size 1.27 1.27)
+			)
+			(justify left)
+		)
+		(property "Intersheetrefs" "${INTERSHEET_REFS}"
+			(at 236.2418 128.27 0)
 			(hide yes)
 			(show_name no)
@@
 		)
 	)
+	(global_label "LED_CAN"
+		(shape input)
+		(at 222.25 143.51 0)
+		(fields_autoplaced yes)
+		(effects
+			(font
+				(size 1.27 1.27)
+			)
+			(justify left)
+		)
+		(property "Intersheetrefs" "${INTERSHEET_REFS}"
+			(at 233.339 143.51 0)
+			(hide yes)
+			(show_name no)
+			(do_not_autoplace no)
+			(effects
+				(font
+					(size 1.27 1.27)
+				)
+				(justify left)
+			)
+		)
+	)
 	(global_label "MOSI"
 		(shape input)
@@
 		)
 	)
-	(global_label "LED3"
-		(shape input)
-		(at 222.25 176.53 0)
-		(fields_autoplaced yes)
-		(effects
-			(font
-				(size 1.27 1.27)
-			)
-			(justify left)
-		)
-		(property "Intersheetrefs" "${INTERSHEET_REFS}"
-			(at 229.8918 176.53 0)
-			(hide yes)
-			(show_name no)
-			(do_not_autoplace no)
-			(effects
-				(font
-					(size 1.27 1.27)
-				)
-				(justify left)
-			)
-		)
-	)
 	(global_label "SW_4"
 		(shape input)
@@
 			(hide yes)
 			(show_name no)
-			(do_not_autoplace no)
-			(effects
-				(font
-					(size 1.27 1.27)
-				)
-				(justify left)
-			)
-		)
-	)
-	(global_label "LED2"
-		(shape input)
-		(at 222.25 173.99 0)
-		(fields_autoplaced yes)
-		(effects
-			(font
-				(size 1.27 1.27)
-			)
-			(justify left)
-		)
-		(property "Intersheetrefs" "${INTERSHEET_REFS}"
-			(at 229.8918 173.99 0)
-			(hide yes)
-			(show_name no)
