File: boards/DashboardV2.0/EVC Dashboard V2/stlink.kicad_sch (KiCad schematic)
At the start: 0 parts

Commit message: added stlink schematic
Parts:
- added C6: .1uF, Capacitor_SMD:C_0603_1608Metric, symbol Device:C
- added J1: Conn_02x05_Odd_Even, Connector_PinSocket_2.54mm:PinSocket_2x05_P2.54mm_Vertical, symbol Connector_Generic:Conn_02x05_Odd_Even
- added JP1, JP2: Jumper_NO_Small, Jumper:SolderJumper-2_P1.3mm_Open_RoundedPad1.0x1.5mm, symbol dashboard-rescue:Jumper_NO_Small-Device
- added JP3, JP4: Jumper_2_Small_Open, Package_LCC:PLCC-84_29.3x29.3mm_P1.27mm, symbol Jumper:Jumper_2_Small_Open
- added R8: 100K, Resistor_SMD:R_0603_1608Metric, symbol Device:R
- added SW1: SW_Push, Button_Switch_SMD:SW_SPST_B3U-3000P, symbol Switch:SW_Push
- added U7: STLINK-V3MODS, STLINK-V3MODS:MODULE_STLINK-V3MODS, symbol STLINK:STLINK-V3MODS
Connections:
- new net: JP4.1 (A), U7.22 (5V_OPT)
- new net: J1.10 (Pin_10), J1.9 (Pin_9), JP2.2
- new net: J1.7 (Pin_7), J1.8 (Pin_8), JP1.1
- new net: JP3.2 (B), U7.30 (T_VCC)
- new net +3V3: JP1.2, R8.1
- new net +5V: JP2.1, JP3.1 (A), JP4.2 (B)
- new net GND: C6.2, J1.3 (Pin_3), J1.4 (Pin_4), SW1.2, U7.24 (GND), U7.26 (GND2), U7.27 (GND3), U7.29 (GND4), U7.5 (GNDDETECT), U7.8 (GND_2)
- new net JTDI: U7.28 (T_JTDI/NC)
- new net NRST: C6.1, J1.1 (Pin_1), R8.2, SW1.1, U7.31 (T_NRST)
- new net SWCLK: J1.6 (Pin_6), U7.13 (T_JCLK/T_SWCLK)
- new net SWDIO: J1.2 (Pin_2), U7.4 (T_JTMS/T_SWDIO)
- new net SWO: J1.5 (Pin_5), U7.6 (T_JTDO/T_SWO)
- new net VCP_RX: U7.15 (T_VCP_RX)
- new net VCP_TX: U7.12 (T_VCP_TX)
- no-connect marks 0 -> 17
Other:
- note added: "Reset Button"
- note added: "ST Link Connector"
- note added: "any of these bridge pins needed?"

Commit message: minor changes to overvoltage protection + comments
changed overvoltage protection chip wiring to better match application in datasheet, also created 5V unlimit input to separate connected 5V to the 5V running through the board (output from overvoltage circuit). also added comments on overvoltage circuit and stlink regarding confusions
Parts:
- added JP5: Jumper_2_Small_Open, Package_LCC:PLCC-84_29.3x29.3mm_P1.27mm, symbol Jumper:Jumper_2_Small_Open
Connections:
- net at JP3.2 (B), U7.30 (T_VCC): now also JP5.2 (B)
- new net +3.3V: JP5.1 (A)
Other:
- note added: "**new change: connected 3.3V by jumper so we have flexbility"
- note added: "i think the VCC pin is rated for 3.3V but it's connected by jumper to 5V in stefan's schematic with comment "Serves as input for STLink if we need it powered off of board""
- note added: "stlink provides 5V but already have 5V on board? keep open through jumper?"
Changed lines of the file:
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@@
+		)
+	)
+	(text "stlink provides 5V but already have 5V \non board? keep open through jumper?"
+		(exclude_from_sim no)
+		(at 138.43 42.164 0)
+		(effects
+			(font
+				(size 1.27 1.27)
+			)
 		)
 	)
@@
 		)
 	)
+	(text "i think the VCC pin is rated for 3.3V but it's \nconnected by jumper to 5V in stefan's schematic\nwith comment \"Serves as input for STLink\nif we need it powered off of board\""
+		(exclude_from_sim no)
+		(at 121.412 110.236 0)
+		(effects
+			(font
+				(size 1.27 1.27)
+			)
+		)
+	)
+	(text "**new change: connected 3.3V by jumper so we have flexbility"
+		(exclude_from_sim no)
+		(at 120.65 117.094 0)
+		(effects
+			(font
+				(size 1.27 1.27)
+			)
+		)
+	)
 	(junction
 		(at 274.32 60.96)
@@
 	)
 	(junction
+		(at 118.11 92.71)
+		(diameter 0)
+		(color 0 0 0 0)
+	)
+	(junction
 		(at 49.53 90.805)
 		(diameter 0)
@@
 	(wire
 		(pts
+			(xy 110.49 102.87) (xy 118.11 102.87)
+		)
+		(stroke
+			(width 0)
+			(type default)
+		)
+	)
+	(wire
+		(pts
 			(xy 55.88 46.355) (xy 46.355 46.355)
 		)
@@
 	(wire
 		(pts
+			(xy 118.11 92.71) (xy 118.11 97.79)
+		)
+		(stroke
+			(width 0)
+			(type default)
+		)
+	)
+	(wire
+		(pts
+			(xy 118.11 92.71) (xy 132.08 92.71)
+		)
+		(stroke
+			(width 0)
+			(type default)
+		)
+	)
+	(wire
+		(pts
 			(xy 68.58 53.975) (xy 68.58 56.515)
 		)
@@
 	(wire
 		(pts
-			(xy 115.57 92.71) (xy 132.08 92.71)
+			(xy 115.57 92.71) (xy 118.11 92.71)
 		)
 		(stroke
@@
 				(path "/ede78d5d-1d5c-4e8d-a13e-c039265851a9/6f5d190a-dfb3-440b-b244-28b5d4db66b6"
 					(reference "J1")
+					(unit 1)
+				)
+			)
+		)
+	)
+	(symbol
+		(lib_name "+3.3V_1")
+		(lib_id "power:+3.3V")
+		(at 110.49 102.87 0)
+		(unit 1)
+		(body_style 1)
+		(exclude_from_sim no)
+		(in_bom yes)
+		(on_board yes)
+		(in_pos_files yes)
+		(dnp no)
+		(fields_autoplaced yes)
+		(property "Reference" "#PWR012"
+			(at 110.49 106.68 0)
+			(hide yes)
+			(show_name no)
+			(do_not_autoplace no)
+			(effects
+				(font
+					(size 1.27 1.27)
+				)
+			)
+		)
+		(property "Value" "+3.3V"
+			(at 110.49 97.79 0)
+			(show_name no)
+			(do_not_autoplace no)
+			(effects
+				(font
+					(size 1.27 1.27)
+				)
+			)
+		)
+		(property "Footprint" ""
+			(at 110.49 102.87 0)
+			(hide yes)
+			(show_name no)
+			(do_not_autoplace no)
+			(effects
+				(font
+					(size 1.27 1.27)
+				)
+			)
+		)
+		(property "Datasheet" ""
+			(at 110.49 102.87 0)
+			(hide yes)
+			(show_name no)
+			(do_not_autoplace no)
+			(effects
+				(font
+					(size 1.27 1.27)
+				)
+			)
+		)
+		(property "Description" "Power symbol creates a global label with name \"+3.3V\""
+			(at 110.49 102.87 0)
+			(hide yes)
+			(show_name no)
+			(do_not_autoplace no)
+			(effects
+				(font
+					(size 1.27 1.27)
+				)
+			)
+		)
+		(pin "1"
+		)
+		(instances
+			(project "EVC Dashboard V2"
+				(path "/ede78d5d-1d5c-4e8d-a13e-c039265851a9/6f5d190a-dfb3-440b-b244-28b5d4db66b6"
+					(reference "#PWR012")
 					(unit 1)
 				)
@@
 					(unit 1)
 				)
+			)
+		)
+	)
+	(symbol
+		(lib_id "Jumper:Jumper_2_Small_Open")
+		(at 118.11 100.33 90)
+		(unit 1)
+		(body_style 1)
+		(exclude_from_sim no)
+		(in_bom yes)
+		(on_board yes)
+		(in_pos_files yes)
+		(dnp no)
+		(fields_autoplaced yes)
+		(property "Reference" "JP5"
+			(at 119.38 99.0599 90)
+			(show_name no)
+			(do_not_autoplace no)
+			(effects
+				(font
+					(size 1.27 1.27)
+				)
+				(justify right)
+			)
+		)
+		(property "Value" "Jumper_2_Small_Open"
+			(at 119.38 101.5999 90)
+			(show_name no)
+			(do_not_autoplace no)
+			(effects
+				(font
+					(size 1.27 1.27)
+				)
+				(justify right)
+			)
+		)
+		(property "Footprint" "Package_LCC:PLCC-84_29.3x29.3mm_P1.27mm"
+			(at 118.11 100.33 0)
+			(hide yes)
+			(show_name no)
+			(do_not_autoplace no)
+			(effects
+				(font
+					(size 1.27 1.27)
+				)
+			)
+		)
+		(property "Datasheet" ""
+			(at 118.11 100.33 0)
+			(hide yes)
+			(show_name no)
+			(do_not_autoplace no)
+			(effects
+				(font
+					(size 1.27 1.27)
+				)
+			)
+		)
+		(property "Description" "Jumper, 2-pole, small symbol, open"
+			(at 118.11 100.33 0)
+			(hide yes)
+			(show_name no)
+			(do_not_autoplace no)
+			(effects
+				(font
+					(size 1.27 1.27)
+				)
+			)
+		)
+		(pin "1"
+		)
+		(pin "2"
+		)
+		(instances
+			(project "EVC Dashboard V2"
+				(path "/ede78d5d-1d5c-4e8d-a13e-c039265851a9/6f5d190a-dfb3-440b-b244-28b5d4db66b6"
+					(reference "JP5")
+					(unit 1)
+				)
