File: boards/Screenless-Dashboard/MCU.kicad_sch (KiCad schematic)
At the start: 0 parts

Commit message: add mcu, finish for today
Parts:
- added U1: STM32H563RGTx, Package_QFP:LQFP-64_10x10mm_P0.5mm, symbol MCU_ST_STM32H5:STM32H563RGTx
Connections:
- new net: U1.18 (VSS), U1.31 (VSS), U1.47 (VSS), U1.63 (VSS)
Changed lines of the file:
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@@
 		(rev "v1.0")
 		(company "Illini EV Concept")
-		(comment 1 "Uses STM32H563RGT6")
+		(comment 1 "Uses STM32H563RGTx")
 		(comment 2 "1 MB flash, 640 KB SPIRAM")
-		(comment 3 "64 Pin LQFP")
+		(comment 3 "LQFP64 Package")
 	)
-)
