File: boards/IMU/imu_PCBv1/imu_PCBv1.kicad_pcb (KiCad board)
At the start: 2 copper layers, 32 parts, among them J1 Debug_Pins, J2 SWD_Header, J4 Micro_SD_Card_Det1, J5 UART, J6 CAN_Bus, J7 USB_C_Receptacle_PowerOnly_6P, U1 ISM330DLCTR, U2 STM32F103RBT6, U4 AP2112K-3.3, U5 ISO1042BQDWQ1, Y1 8MHz

Commit message: First draft of IMU layout
Parts:
- removed J1: Debug_Pins, Connector_PinHeader_2.54mm:PinHeader_1x10_P2.54mm_Vertical
- added J3: Conn_01x08_Pin, Connector_PinHeader_2.54mm:PinHeader_1x08_P2.54mm_Vertical, F.Cu at (158.3, 82.0)
- moved C15 47.1 mm to (186.0, 97.5), turned to 180 degrees
- moved R8 46.9 mm to (188.0, 89.5), turned to 90 degrees
- moved C12 41.7 mm to (179.5, 88.0), turned to 90 degrees
- moved J6 39.2 mm to (184.0, 112.5)
- moved R3 38.5 mm to (183.6, 94.0)
- moved C4 37.4 mm to (170.0, 89.5), turned to -90 degrees
- moved R2 33.9 mm to (155.4, 86.0), turned to 180 degrees
- moved C11 32.0 mm to (172.0, 93.5)
- moved J5 28.8 mm to (143.9, 104.6)
- moved C3 28.8 mm to (165.5, 105.5), turned to 90 degrees
- moved U2 28.4 mm to (162.0, 96.5)
- moved Y1 28.4 mm to (148.0, 92.2)
- moved R4 28.3 mm to (172.5, 110.0), turned to 90 degrees
- moved J7 28.1 mm to (194.0, 90.3), turned to 90 degrees
- moved C5 26.3 mm to (152.3, 88.0)
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Connections:
- U2 pad 10: /GPIO_2 -> unconnected-(U2-PC2-Pad10)
- U2 pad 11: /GPIO_3 -> unconnected-(U2-PC3-Pad11)
- U2 pad 24: /GPIO_4 -> unconnected-(U2-PC4-Pad24)
- U2 pad 25: /GPIO_5 -> unconnected-(U2-PC5-Pad25)
- U2 pad 37: /GPIO_6 -> unconnected-(U2-PC6-Pad37)
- U2 pad 38: /GPIO_7 -> unconnected-(U2-PC7-Pad38)
- U2 pad 39: /GPIO_8 -> unconnected-(U2-PC8-Pad39)
- U2 pad 40: /GPIO_9 -> unconnected-(U2-PC9-Pad40)
- U2 pad 50: unconnected-(U2-PA15-Pad50) -> /GPIO_8
- U2 pad 51: /GPIO_10 -> /GPIO_7
- U2 pad 52: unconnected-(U2-PC11-Pad52) -> /GPIO_6
- U2 pad 53: unconnected-(U2-PC12-Pad53) -> /GPIO_5
- U2 pad 54: unconnected-(U2-PD2-Pad54) -> /GPIO_4
- U2 pad 55: unconnected-(U2-PB3-Pad55) -> /GPIO_3
- U2 pad 56: unconnected-(U2-PB4-Pad56) -> /GPIO_2
- U2 pad 57: unconnected-(U2-PB5-Pad57) -> /GPIO_1
- U2 pad 9: /GPIO_1 -> unconnected-(U2-PC1-Pad9)
Routing:
- net GND: track 0.00 -> 136.2 mm, vias 0 -> 16
- net 3.3V: track 0.00 -> 81.8 mm, vias 0 -> 2
- net /NRST: track 0.00 -> 47.7 mm, vias 0 -> 2
- net /INT1: track 0.00 -> 35.5 mm, vias 0 -> 2
- net /USB_VIN: track 0.00 -> 33.6 mm
- net /SWDIO: track 0.00 -> 26.7 mm
- net /DET: track 0.00 -> 26.1 mm, vias 0 -> 2
- net Net-(J4-DAT0): track 0.00 -> 24.1 mm, vias 0 -> 2
- net Net-(J4-CMD): track 0.00 -> 23.6 mm, vias 0 -> 2
- net /SWCLK: track 0.00 -> 20.8 mm
- net /CS: track 0.00 -> 20.3 mm
- net Net-(J4-DAT3/CD): track 0.00 -> 19.4 mm, vias 0 -> 2
- net Net-(J4-CLK): track 0.00 -> 17.3 mm
- net /GPIO_8: track 0.00 -> 14.9 mm
- net /CANH: track 0.00 -> 13.5 mm
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- added copper zone on F.Cu, net 3.3V
- added copper zone on B.Cu, net GND
